Commit message: add temp sens global map

File: src/ursa/urdf/ursa.urdf (robot description, URDF)
Before this commit: robot ursa, 6 links, 5 joints
Links:
- added link temp_link; visual cylinder length=0.05 radius=0.03
Joints:
- added joint temp_link_joint: type fixed, parent base_link, child temp_link, origin xyz=-0.12 0 0 rpy=0 0 -0.131

Commit message: Enable move base with new Carto

File: src/ursa/urdf/ursa.urdf (robot description, URDF)
Before this commit: robot ursa, 7 links, 6 joints
Links:
- removed link temp_link
Joints:
- removed joint temp_link_joint
